Commit message: 新文件：   events.out.tfevents.1712255520.dhu423a-Precision-7920-Tower.19304.0 	修改：     resources/robots/wl/CMakeLists.txt 	新文件：   resources/robots/wl/config/joint_names_wl-4.yaml 	修改：     resources/robots/wl/launch/display.launch 	修改：     resources/robots/wl/launch/gazebo.launch 	修改：     resources/robots/wl/meshes/base_link.STL 	修改：     resources/robots/wl/meshes/l_wheel_Link.STL 	修改：     resources/robots/wl/meshes/lf0_Link.STL 	修改：     resources/robots/wl/meshes/lf1_Link.STL 	修改：     resources/robots/wl/meshes/r_wheel_Link.STL 	修改：     resources/robots/wl/meshes/rf0_Link.STL 	修改：     resources/robots/wl/meshes/rf1_Link.STL 	修改：     resources/robots/wl/package.xml 	修改：     resources/robots/wl/urdf/wl.csv 	修改：     resources/robots/wl/urdf/wl.urdf 	新文件：   resources/wl-1/CMakeLists.txt 	重命名：   resources/robots/wl/config/joint_names_wheel_legged_open.yaml -> resources/wl-1/config/joint_names_wheel_legged_open.yaml 	新文件：   resources/wl-1/launch/display.launch 	新文件：   resources/wl-1/launch/gazebo.launch 	新文件：   resources/wl-1/meshes/base_link.STL 	新文件：   resources/wl-1/meshes/l_wheel_Link.STL 	新文件：   resources/wl-1/meshes/lf0_Link.STL 	新文件：   resources/wl-1/meshes/lf1_Link.STL 	新文件：   resources/wl-1/meshes/r_wheel_Link.STL 	新文件：   resources/wl-1/meshes/rf0_Link.STL 	新文件：   resources/wl-1/meshes/rf1_Link.STL 	新文件：   resources/wl-1/package.xml 	新文件：   resources/wl-1/urdf/wl.csv 	新文件：   resources/wl-1/urdf/wl.urdf 	新文件：   resources/wl/CMakeLists.txt 	新文件：   resources/wl/config/joint_names_wl-4.yaml 	新文件：   resources/wl/launch/display.launch 	新文件：   resources/wl/launch/gazebo.launch 	新文件：   resources/wl/meshes/base_link.STL 	新文件：   resources/wl/meshes/l_wheel_Link.STL 	新文件：   resources/wl/meshes/lf0_Link.STL 	新文件：   resources/wl/meshes/lf1_Link.STL 	新文件：   resources/wl/meshes/r_wheel_Link.STL 	新文件：   resources/wl/meshes/rf0_Link.STL 	新文件：   resources/wl/meshes/rf1_Link.STL 	新文件：   resources/wl/package.xml 	新文件：   resources/wl/urdf/wl-4.csv 	新文件：   resources/wl/urdf/wl-4.urdf 	修改：     wheel_legged_gym/scripts/play.py 	修改：     wheel_legged_gym/scripts/train.py 	修改：     wheel_legged_gym/utils/__init__.py 	新文件：   wheel_legged_gym/utils/exporter.py 	修改：     wheel_legged_gym/utils/helpers.py

File: resources/wl/urdf/wl-4.urdf (robot description, URDF)
Before this commit: robot wl-4, 7 links, 6 joints
Links:
- link base_link: geometry collision mesh filename=package://wl-4/meshes/base_link.STL; visual mesh filename=package://wl-4/meshes/base_link.STL
- link l_wheel_Link: geometry collision mesh filename=package://wl-4/meshes/l_wheel_Link.STL; visual mesh filename=package://wl-4/meshes/l_wheel_Link.STL
- link lf0_Link: geometry collision mesh filename=package://wl-4/meshes/lf0_Link.STL; visual mesh filename=package://wl-4/meshes/lf0_Link.STL
- link lf1_Link: geometry collision mesh filename=package://wl-4/meshes/lf1_Link.STL; visual mesh filename=package://wl-4/meshes/lf1_Link.STL
- link r_wheel_Link: geometry collision mesh filename=package://wl-4/meshes/r_wheel_Link.STL; visual mesh filename=package://wl-4/meshes/r_wheel_Link.STL
- link rf0_Link: geometry collision mesh filename=package://wl-4/meshes/rf0_Link.STL; visual mesh filename=package://wl-4/meshes/rf0_Link.STL
- link rf1_Link: geometry collision mesh filename=package://wl-4/meshes/rf1_Link.STL; visual mesh filename=package://wl-4/meshes/rf1_Link.STL
Joints:
- joint l_wheel_Joint: type revolute -> continuous
- joint lf0_Joint: limit lower=-1.3479 upper=-0.35 effort=30 velocity=1000 -> lower=-0.2182 upper=1.3479 effort=30 velocity=1000; type revolute -> continuous
- joint lf1_Joint: limit lower=-2.0 upper=0 effort=30 velocity=1000 -> lower=-1 upper=1.25 effort=30 velocity=1000; type revolute -> continuous
- joint r_wheel_Joint: type revolute -> continuous
- joint rf0_Joint: limit lower=0.35 upper=1.3479 effort=30 velocity=1000 -> lower=-0.2182 upper=1.3479 effort=30 velocity=1000; type revolute -> continuous
- joint rf1_Joint: limit lower=0 upper=2.0 effort=30 velocity=1000 -> lower=-1 upper=1.25 effort=30 velocity=1000; type revolute -> continuous
