Commit message: 重命名：   resources/wl-1/CMakeLists.txt -> resources/robots/wl-1/CMakeLists.txt 	重命名：   resources/wl-1/config/joint_names_wheel_legged_open.yaml -> resources/robots/wl-1/config/joint_names_wheel_legged_open.yaml 	重命名：   resources/wl-1/launch/display.launch -> resources/robots/wl-1/launch/display.launch 	重命名：   resources/wl-1/launch/gazebo.launch -> resources/robots/wl-1/launch/gazebo.launch 	重命名：   resources/wl-1/meshes/base_link.STL -> resources/robots/wl-1/meshes/base_link.STL 	重命名：   resources/wl-1/meshes/l_wheel_Link.STL -> resources/robots/wl-1/meshes/l_wheel_Link.STL 	重命名：   resources/wl-1/meshes/lf0_Link.STL -> resources/robots/wl-1/meshes/lf0_Link.STL 	重命名：   resources/wl-1/meshes/lf1_Link.STL -> resources/robots/wl-1/meshes/lf1_Link.STL 	重命名：   resources/wl-1/meshes/r_wheel_Link.STL -> resources/robots/wl-1/meshes/r_wheel_Link.STL 	重命名：   resources/wl-1/meshes/rf0_Link.STL -> resources/robots/wl-1/meshes/rf0_Link.STL 	重命名：   resources/wl-1/meshes/rf1_Link.STL -> resources/robots/wl-1/meshes/rf1_Link.STL 	重命名：   resources/wl-1/package.xml -> resources/robots/wl-1/package.xml 	重命名：   resources/wl-1/urdf/wl.csv -> resources/robots/wl-1/urdf/wl.csv 	重命名：   resources/wl-1/urdf/wl.urdf -> resources/robots/wl-1/urdf/wl.urdf 	修改：     resources/robots/wl/CMakeLists.txt 	重命名：   resources/robots/wl/config/joint_names_wl-4.yaml -> resources/robots/wl/config/joint_names_wl.yaml 	修改：     resources/robots/wl/launch/display.launch 	修改：     resources/robots/wl/launch/gazebo.launch 	修改：     resources/robots/wl/meshes/base_link.STL 	修改：     resources/robots/wl/meshes/l_wheel_Link.STL 	修改：     resources/robots/wl/meshes/lf0_Link.STL 	修改：     resources/robots/wl/meshes/lf1_Link.STL 	修改：     resources/robots/wl/meshes/r_wheel_Link.STL 	修改：     resources/robots/wl/meshes/rf0_Link.STL 	修改：     resources/robots/wl/meshes/rf1_Link.STL 	修改：     resources/robots/wl/package.xml 	修改：     resources/robots/wl/urdf/wl.csv 	修改：     resources/robots/wl/urdf/wl.urdf 	修改：     wheel_legged_gym/envs/wheel_legged/wheel_legged_config.py 	修改：     wheel_legged_gym/envs/wheel_legged_vmc/wheel_legged_vmc.py 	修改：     wheel_legged_gym/envs/wheel_legged_vmc/wheel_legged_vmc_config.py 	修改：     wheel_legged_gym/envs/wheel_legged_vmc_flat/wheel_legged_vmc_flat_config.py 	修改：     wheel_legged_gym/scripts/play.py 	修改：     wheel_legged_gym/scripts/train.py

File: resources/robots/wl/urdf/wl.urdf (robot description, URDF)
Before this commit: robot wl-4, 7 links, 6 joints
Links:
- link base_link: mass 2.2729 -> 2.7026
Joints:
- joint l_wheel_Joint: axis 1 0 0 -> 0 0 1; limit effort=5 velocity=1000 -> lower=0 upper=0 effort=60 velocity=1000; origin xyz=-0.046511 -0.12948 -0.20207 rpy=-0.10149 0 -3.1416 -> xyz=-0.22699 -0.077958 0.014 rpy=-3.1416 0 0
- joint lf0_Joint: axis 1 0 0 -> 0 0 -1; limit lower=-1.3479 upper=-0.35 effort=30 velocity=1000 -> lower=0.44 upper=1.3962 effort=50 velocity=1000; origin xyz=-0.048289 -0.23 0.045 rpy=-1.1943 0 -3.1416 -> xyz=-0.055 0.1793 0.054 rpy=1.5708 0 3.1416
- joint lf1_Joint: axis 1 0 0 -> 0 0 -1; limit lower=-2.0 upper=0 effort=30 velocity=1000 -> lower=-2.7925 upper=-0.44 effort=50 velocity=1000; origin xyz=0 0.029484 0.14707 rpy=0.26553 0 3.1416 -> xyz=0.15 0 0.033 rpy=0 0 0
- joint r_wheel_Joint: limit effort=5 velocity=1000 -> lower=0 upper=0 effort=5 velocity=1000; origin xyz=-0.053011 -0.12948 -0.20207 rpy=1.5708 0.32015 -1.5708 -> xyz=0.22699 -0.077958 0.0135 rpy=0 0 3.1416
- joint rf0_Joint: axis 1 0 0 -> 0 0 1; limit lower=0.35 upper=1.3479 effort=30 velocity=1000 -> lower=0.44 upper=1.3962 effort=50 velocity=1000; origin xyz=0.29829 -0.23 0.045 rpy=1.59 0 0 -> xyz=-0.055 -0.1793 0.054 rpy=1.5708 0 0
- joint rf1_Joint: axis 1 0 0 -> 0 0 -1; limit lower=0 upper=2.0 effort=30 velocity=1000 -> lower=0.44 upper=2.7925 effort=50 velocity=1000; origin xyz=0 0.029484 0.14707 rpy=1.2699 0 -3.1416 -> xyz=-0.15 0 0.0335 rpy=0 0 0
